File: board/RAMBo.sch (EAGLE design)
At the start: 266 parts, among them Q1 PSMN7R0-60YS, Q2 PSMN7R0-60YS, Q3 PSMN7R0-60YS, Q4 IRLML6346TRPBF, Q5 PSMN7R0-60YS, Q8 IRLML6346TRPBF, U1 ATMEGA32U2-MUR, U10 ADUM7441, U2 ATMEGA2560-16AU, U3 LM22675, U4 AD5206, U5 A4982, U6 A4982, U7 A4982, U8 A4982, U9 A4982, X1 C-GRID-02-70543, X10 C-GRID-04-70543, X11 MSTBV10, X12 SPI, X13 EXT-2, X14 C-GRID-04-70543, X15 C-GRID-04-70543, X16 32u2 EXT, X17 3x2M, X18 3x2M, X2 USB B-TH, X20 MX1, X21 C-GRID-03-70543, X22 C-GRID-03-70543, X23 C-GRID-03-70543, X24 C-GRID-03-70543, X25 C-GRID-03-70543, X26 C-GRID-03-70543, X27 C-GRID-02-70543, X28 C-GRID-02-70543, X29 C-GRID-02-70543, X3 C-GRID-02-70543, X30 C-GRID-02-70543, X31 MX2, X32 MX3, X33 MSTBA6, X34 PWM_EXT, X39 M05X2PTH, X4 C-GRID-04-70543, X40 Analog, X5 C-GRID-02-70543, X6 C-GRID-04-70543, X7 C-GRID-04-70543, X8 C-GRID-04-70543, X9 C-GRID-02-70543, Y1 16MHz KX-7, Y2 16MHz KX-7

Commit message: Clean up schematic, publish pdf in docs
Other:
- note added: "Atmega2560 Programmer"
- note added: "I2C Expansion"
- note added: "Insert jumper to disable on-board PSU"
- note added: "RAMBo 1.2e"
- note added: "Stepper Motor Drivers"
- note removed: "3SMAJ5938B-TP on motors for overvoltage cap @ 36V"
- note removed: "Atmega2560 programmer"
- note removed: "I2C expansion"
- note removed: "Logic Power Select"
- note removed: "Rambo 1.2"
- note removed: "Stepper motor drivers"
- moved on the sheet: C7, C8, C9, D3, H1, H2, H3

Commit message: change stepper test points to through hole
YEN, ZDIR, and E0DIR moved to clear bottom traces
Parts:
- TP0, TP1, TP10, TP11, TP12, TP13, TP14, TP15, TP16, TP17, TP18, TP19, TP2, TP3, TP4, TP5, TP6, TP7, TP8, TP9: value PTR1B1,27 -> PTR1B1,27TH; device testpad:PTR1B1,27 -> testpad:PTR1B1,27TH
Changed lines of the file:
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@@
 <grid distance="0.1" unitdist="inch" unit="inch" style="lines" multiple="1" display="no" altdistance="0.01" altunitdist="inch" altunit="inch"/>
 <layers>
-<layer number="1" name="Top" color="4" fill="1" visible="yes" active="no"/>
-<layer number="2" name="Route2" color="13" fill="3" visible="yes" active="no"/>
-<layer number="3" name="Route3" color="4" fill="3" visible="yes" active="no"/>
-<layer number="14" name="Route14" color="1" fill="6" visible="yes" active="no"/>
-<layer number="15" name="Route15" color="11" fill="6" visible="yes" active="no"/>
-<layer number="16" name="Bottom" color="1" fill="1" visible="yes" active="no"/>
-<layer number="17" name="Pads" color="2" fill="1" visible="yes" active="no"/>
-<layer number="18" name="Vias" color="2" fill="1" visible="yes" active="no"/>
-<layer number="19" name="Unrouted" color="6" fill="1" visible="yes" active="no"/>
-<layer number="20" name="Dimension" color="15" fill="1" visible="yes" active="no"/>
-<layer number="21" name="tPlace" color="7" fill="1" visible="yes" active="no"/>
-<layer number="22" name="bPlace" color="7" fill="1" visible="yes" active="no"/>
-<layer number="23" name="tOrigins" color="15" fill="1" visible="yes" active="no"/>
-<layer number="24" name="bOrigins" color="15" fill="1" visible="yes" active="no"/>
-<layer number="25" name="tNames" color="7" fill="1" visible="yes" active="no"/>
-<layer number="26" name="bNames" color="7" fill="1" visible="yes" active="no"/>
-<layer number="27" name="tValues" color="7" fill="1" visible="yes" active="no"/>
-<layer number="28" name="bValues" color="7" fill="1" visible="yes" active="no"/>
+<layer number="1" name="Top" color="4" fill="1" visible="no" active="no"/>
+<layer number="2" name="Route2" color="13" fill="3" visible="no" active="no"/>
+<layer number="3" name="Route3" color="4" fill="3" visible="no" active="no"/>
+<layer number="14" name="Route14" color="1" fill="6" visible="no" active="no"/>
+<layer number="15" name="Route15" color="11" fill="6" visible="no" active="no"/>
+<layer number="16" name="Bottom" color="1" fill="1" visible="no" active="no"/>
+<layer number="17" name="Pads" color="2" fill="1" visible="no" active="no"/>
+<layer number="18" name="Vias" color="2" fill="1" visible="no" active="no"/>
+<layer number="19" name="Unrouted" color="6" fill="1" visible="no" active="no"/>
+<layer number="20" name="Dimension" color="15" fill="1" visible="no" active="no"/>
+<layer number="21" name="tPlace" color="7" fill="1" visible="no" active="no"/>
+<layer number="22" name="bPlace" color="7" fill="1" visible="no" active="no"/>
+<layer number="23" name="tOrigins" color="15" fill="1" visible="no" active="no"/>
+<layer number="24" name="bOrigins" color="15" fill="1" visible="no" active="no"/>
+<layer number="25" name="tNames" color="7" fill="1" visible="no" active="no"/>
+<layer number="26" name="bNames" color="7" fill="1" visible="no" active="no"/>
+<layer number="27" name="tValues" color="7" fill="1" visible="no" active="no"/>
+<layer number="28" name="bValues" color="7" fill="1" visible="no" active="no"/>
 <layer number="29" name="tStop" color="7" fill="3" visible="no" active="no"/>
 <layer number="30" name="bStop" color="7" fill="6" visible="no" active="no"/>
@@
 <layer number="35" name="tGlue" color="7" fill="4" visible="no" active="no"/>
 <layer number="36" name="bGlue" color="7" fill="5" visible="no" active="no"/>
-<layer number="37" name="tTest" color="7" fill="1" visible="yes" active="no"/>
-<layer number="38" name="bTest" color="7" fill="1" visible="yes" active="no"/>
+<layer number="37" name="tTest" color="7" fill="1" visible="no" active="no"/>
+<layer number="38" name="bTest" color="7" fill="1" visible="no" active="no"/>
 <layer number="39" name="tKeepout" color="4" fill="11" visible="no" active="no"/>
 <layer number="40" name="bKeepout" color="1" fill="11" visible="no" active="no"/>
@@
 <layer number="44" name="Drills" color="7" fill="1" visible="no" active="no"/>
 <layer number="45" name="Holes" color="7" fill="1" visible="no" active="no"/>
-<layer number="46" name="Milling" color="3" fill="1" visible="yes" active="no"/>
-<layer number="47" name="Measures" color="7" fill="1" visible="yes" active="no"/>
-<layer number="48" name="Document" color="7" fill="1" visible="yes" active="no"/>
-<layer number="49" name="Reference" color="7" fill="1" visible="yes" active="no"/>
-<layer number="50" name="dxf" color="12" fill="1" visible="yes" active="no"/>
-<layer number="51" name="tDocu" color="7" fill="1" visible="yes" active="no"/>
-<layer number="52" name="bDocu" color="7" fill="1" visible="yes" active="no"/>
-<layer number="53" name="tGND_GNDA" color="7" fill="1" visible="yes" active="no"/>
-<layer number="54" name="bGND_GNDA" color="7" fill="1" visible="yes" active="no"/>
-<layer number="56" name="wert" color="7" fill="1" visible="yes" active="no"/>
+<layer number="46" name="Milling" color="3" fill="1" visible="no" active="no"/>
+<layer number="47" name="Measures" color="7" fill="1" visible="no" active="no"/>
+<layer number="48" name="Document" color="7" fill="1" visible="no" active="no"/>
+<layer number="49" name="Reference" color="7" fill="1" visible="no" active="no"/>
+<layer number="50" name="dxf" color="12" fill="1" visible="no" active="no"/>
+<layer number="51" name="tDocu" color="7" fill="1" visible="no" active="no"/>
+<layer number="52" name="bDocu" color="7" fill="1" visible="no" active="no"/>
+<layer number="53" name="tGND_GNDA" color="7" fill="1" visible="no" active="no"/>
+<layer number="54" name="bGND_GNDA" color="7" fill="1" visible="no" active="no"/>
+<layer number="56" name="wert" color="7" fill="1" visible="no" active="no"/>
 <layer number="91" name="Nets" color="2" fill="1" visible="yes" active="yes"/>
 <layer number="92" name="Busses" color="1" fill="1" visible="yes" active="yes"/>
@@
 <part name="X1" library="con-molex" deviceset="C-GRID-02" device="-70543" value="C-GRID-02-70543"/>
 <part name="GND7" library="supply1" deviceset="GND" device=""/>
-<part name="TP3" library="testpad" deviceset="PTR1" device="B1,27"/>
-<part name="TP2" library="testpad" deviceset="PTR1" device="B1,27"/>
-<part name="TP1" library="testpad" deviceset="PTR1" device="B1,27"/>
-<part name="TP4" library="testpad" deviceset="PTR1" device="B1,27"/>
-<part name="TP6" library="testpad" deviceset="PTR1" device="B1,27"/>
-<part name="TP5" library="testpad" deviceset="PTR1" device="B1,27"/>
-<part name="TP0" library="testpad" deviceset="PTR1" device="B1,27"/>
-<part name="TP7" library="testpad" deviceset="PTR1" device="B1,27"/>
-<part name="TP9" library="testpad" deviceset="PTR1" device="B1,27"/>
-<part name="TP8" library="testpad" deviceset="PTR1" device="B1,27"/>
-<part name="TP19" library="testpad" deviceset="PTR1" device="B1,27"/>
-<part name="TP10" library="testpad" deviceset="PTR1" device="B1,27"/>
-<part name="TP12" library="testpad" deviceset="PTR1" device="B1,27"/>
-<part name="TP13" library="testpad" deviceset="PTR1" device="B1,27"/>
-<part name="TP11" library="testpad" deviceset="PTR1" device="B1,27"/>
-<part name="TP14" library="testpad" deviceset="PTR1" device="B1,27"/>
-<part name="TP17" library="testpad" deviceset="PTR1" device="B1,27"/>
-<part name="TP16" library="testpad" deviceset="PTR1" device="B1,27"/>
-<part name="TP15" library="testpad" deviceset="PTR1" device="B1,27"/>
-<part name="TP18" library="testpad" deviceset="PTR1" device="B1,27"/>
+<part name="TP3" library="testpad" deviceset="PTR1" device="B1,27TH" value="PTR1B1,27TH"/>
+<part name="TP2" library="testpad" deviceset="PTR1" device="B1,27TH" value="PTR1B1,27TH"/>
+<part name="TP1" library="testpad" deviceset="PTR1" device="B1,27TH" value="PTR1B1,27TH"/>
+<part name="TP4" library="testpad" deviceset="PTR1" device="B1,27TH" value="PTR1B1,27TH"/>
+<part name="TP6" library="testpad" deviceset="PTR1" device="B1,27TH" value="PTR1B1,27TH"/>
+<part name="TP5" library="testpad" deviceset="PTR1" device="B1,27TH" value="PTR1B1,27TH"/>
+<part name="TP0" library="testpad" deviceset="PTR1" device="B1,27TH" value="PTR1B1,27TH"/>
+<part name="TP7" library="testpad" deviceset="PTR1" device="B1,27TH" value="PTR1B1,27TH"/>
+<part name="TP9" library="testpad" deviceset="PTR1" device="B1,27TH" value="PTR1B1,27TH"/>
+<part name="TP8" library="testpad" deviceset="PTR1" device="B1,27TH" value="PTR1B1,27TH"/>
+<part name="TP19" library="testpad" deviceset="PTR1" device="B1,27TH" value="PTR1B1,27TH"/>
+<part name="TP10" library="testpad" deviceset="PTR1" device="B1,27TH" value="PTR1B1,27TH"/>
+<part name="TP12" library="testpad" deviceset="PTR1" device="B1,27TH" value="PTR1B1,27TH"/>
+<part name="TP13" library="testpad" deviceset="PTR1" device="B1,27TH" value="PTR1B1,27TH"/>
+<part name="TP11" library="testpad" deviceset="PTR1" device="B1,27TH" value="PTR1B1,27TH"/>
+<part name="TP14" library="testpad" deviceset="PTR1" device="B1,27TH" value="PTR1B1,27TH"/>
+<part name="TP17" library="testpad" deviceset="PTR1" device="B1,27TH" value="PTR1B1,27TH"/>
+<part name="TP16" library="testpad" deviceset="PTR1" device="B1,27TH" value="PTR1B1,27TH"/>
+<part name="TP15" library="testpad" deviceset="PTR1" device="B1,27TH" value="PTR1B1,27TH"/>
+<part name="TP18" library="testpad" deviceset="PTR1" device="B1,27TH" value="PTR1B1,27TH"/>
 <part name="TP22" library="testpad" deviceset="PTR1" device="B1,27"/>
 <part name="TP21" library="testpad" deviceset="PTR1" device="B1,27"/>
